Commit message: new file:   robotiq_85_gripper/LICENSE 	new file:   robotiq_85_gripper/README.md 	new file:   robotiq_85_gripper/robotiq_85_bringup/CMakeLists.txt 	new file:   robotiq_85_gripper/robotiq_85_bringup/launch/robotiq_85.launch 	new file:   robotiq_85_gripper/robotiq_85_bringup/package.xml 	new file:   robotiq_85_gripper/robotiq_85_bringup/rviz/robotiq_85.rviz 	new file:   robotiq_85_gripper/robotiq_85_description/CMakeLists.txt 	new file:   robotiq_85_gripper/robotiq_85_description/launch/display.launch 	new file:   robotiq_85_gripper/robotiq_85_description/launch/upload_robotiq_85_gripper.launch 	new file:   robotiq_85_gripper/robotiq_85_description/meshes/collision/kinova_robotiq_coupler.stl 	new file:   robotiq_85_gripper/robotiq_85_description/meshes/collision/robotiq_85_base_link.stl 	new file:   robotiq_85_gripper/robotiq_85_description/meshes/collision/robotiq_85_finger_link.stl 	new file:   robotiq_85_gripper/robotiq_85_description/meshes/collision/robotiq_85_finger_tip_link.stl 	new file:   robotiq_85_gripper/robotiq_85_description/meshes/collision/robotiq_85_inner_knuckle_link.stl 	new file:   robotiq_85_gripper/robotiq_85_description/meshes/collision/robotiq_85_knuckle_link.stl 	new file:   robotiq_85_gripper/robotiq_85_description/meshes/visual/kinova_robotiq_coupler.dae 	new file:   robotiq_85_gripper/robotiq_85_description/meshes/visual/robotiq_85_base_link.dae 	new file:   robotiq_85_gripper/robotiq_85_description/meshes/visual/robotiq_85_finger_link.dae 	new file:   robotiq_85_gripper/robotiq_85_description/meshes/visual/robotiq_85_finger_tip_link.dae 	new file:   robotiq_85_gripper/robotiq_85_description/meshes/visual/robotiq_85_inner_knuckle_link.dae 	new file:   robotiq_85_gripper/robotiq_85_description/meshes/visual/robotiq_85_knuckle_link.dae 	new file:   robotiq_85_gripper/robotiq_85_description/package.xml 	new file:   robotiq_85_gripper/robotiq_85_description/urdf.rviz 	new file:   robotiq_85_gripper/robotiq_85_description/urdf/kinova_robotiq_85_gripper.xacro 	new file:   robotiq_85_gripper/robotiq_85_description/urdf/robotiq_85_gripper.transmission.xacro 	new file:   robotiq_85_gripper/robotiq_85_description/urdf/robotiq_85_gripper.urdf.xacro 	new file:   robotiq_85_gripper/robotiq_85_description/urdf/robotiq_85_gripper.xacro 	new file:   robotiq_85_gripper/robotiq_85_description/urdf/robotiq_85_gripper_sim_base.urdf.xacro 	new file:   robotiq_85_gripper/robotiq_85_description/urdf/robotiq_85_kinova_coupler.urdf.xacro 	new file:   robotiq_85_gripper/robotiq_85_driver/CMakeLists.txt 	new file:   robotiq_85_gripper/robotiq_85_driver/bin/robotiq_85_driver 	new file:   robotiq_85_gripper/robotiq_85_driver/bin/robotiq_85_test 	new file:   robotiq_85_gripper/robotiq_85_driver/package.xml 	new file:   robotiq_85_gripper/robotiq_85_driver/setup.py 	new file:   robotiq_85_gripper/robotiq_85_driver/src/robotiq_85/__init__.py 	new file:   robotiq_85_gripper/robotiq_85_driver/src/robotiq_85/gripper_io.py 	new file:   robotiq_85_gripper/robotiq_85_driver/src/robotiq_85/modbus_crc.py 	new file:   robotiq_85_gripper/robotiq_85_driver/src/robotiq_85/robotiq_85_driver.py 	new file:   robotiq_85_gripper/robotiq_85_driver/src/robotiq_85/robotiq_85_gripper.py 	new file:   robotiq_85_gripper/robotiq_85_driver/src/robotiq_85/robotiq_85_gripper_test.py 	new file:   robotiq_85_gripper/robotiq_85_gripper/CMakeLists.txt 	new file:   robotiq_85_gripper/robotiq_85_gripper/package.xml 	new file:   robotiq_85_gripper/robotiq_85_moveit_config/.setup_assistant 	new file:   robotiq_85_gripper/robotiq_85_moveit_config/CMakeLists.txt 	new file:   robotiq_85_gripper/robotiq_85_moveit_config/config/controllers.yaml 	new file:   robotiq_85_gripper/robotiq_85_moveit_config/config/fake_controllers.yaml 	new file:   robotiq_85_gripper/robotiq_85_moveit_config/config/joint_limits.yaml 	new file:   robotiq_85_gripper/robotiq_85_moveit_config/config/kinematics.yaml 	new file:   robotiq_85_gripper/robotiq_85_moveit_config/config/ompl_planning.yaml 	new file:   robotiq_85_gripper/robotiq_85_moveit_config/config/robotiq_85_gripper.srdf 	new file:   robotiq_85_gripper/robotiq_85_moveit_config/launch/default_warehouse_db.launch 	new file:   robotiq_85_gripper/robotiq_85_moveit_config/launch/demo.launch 	new file:   robotiq_85_gripper/robotiq_85_moveit_config/launch/fake_moveit_controller_manager.launch.xml 	new file:   robotiq_85_gripper/robotiq_85_moveit_config/launch/joystick_control.launch 	new file:   robotiq_85_gripper/robotiq_85_moveit_config/launch/move_group.launch 	new file:   robotiq_85_gripper/robotiq_85_moveit_config/launch/moveit.rviz 	new file:   robotiq_85_gripper/robotiq_85_moveit_config/launch/moveit_rviz.launch 	new file:   robotiq_85_gripper/robotiq_85_moveit_config/launch/ompl_planning_pipeline.launch.xml 	new file:   robotiq_85_gripper/robotiq_85_moveit_config/launch/planning_context.launch 	new file:   robotiq_85_gripper/robotiq_85_moveit_config/launch/planning_pipeline.launch.xml 	new file:   robotiq_85_gripper/robotiq_85_moveit_config/launch/robotiq_85_gripper_moveit_controller_manager.launch.xml 	new file:   robotiq_85_gripper/robotiq_85_moveit_config/launch/robotiq_85_gripper_moveit_sensor_manager.launch.xml 	new file:   robotiq_85_gripper/robotiq_85_moveit_config/launch/robotiq_85_moveit_planning_execution.launch 	new file:   robotiq_85_gripper/robotiq_85_moveit_config/launch/run_benchmark_ompl.launch 	new file:   robotiq_85_gripper/robotiq_85_moveit_config/launch/sensor_manager.launch.xml 	new file:   robotiq_85_gripper/robotiq_85_moveit_config/launch/setup_assistant.launch 	new file:   robotiq_85_gripper/robotiq_85_moveit_config/launch/trajectory_execution.launch.xml 	new file:   robotiq_85_gripper/robotiq_85_moveit_config/launch/warehouse.launch 	new file:   robotiq_85_gripper/robotiq_85_moveit_config/launch/warehouse_settings.launch.xml 	new file:   robotiq_85_gripper/robotiq_85_moveit_config/package.xml 	new file:   robotiq_85_gripper/robotiq_85_msgs/CMakeLists.txt 	new file:   robotiq_85_gripper/robotiq_85_msgs/msg/GripperCmd.msg 	new file:   robotiq_85_gripper/robotiq_85_msgs/msg/GripperStat.msg 	new file:   robotiq_85_gripper/robotiq_85_msgs/package.xml 	new file:   robotiq_85_gripper/robotiq_85_simulation/roboticsgroup_gazebo_plugins/CMakeLists.txt 	new file:   robotiq_85_gripper/robotiq_85_simulation/roboticsgroup_gazebo_plugins/README.md 	new file:   robotiq_85_gripper/robotiq_85_simulation/roboticsgroup_gazebo_plugins/include/roboticsgroup_gazebo_plugins/disable_link_plugin.h 	new file:   robotiq_85_gripper/robotiq_85_simulation/roboticsgroup_gazebo_plugins/include/roboticsgroup_gazebo_plugins/mimic_joint_plugin.h 	new file:   robotiq_85_gripper/robotiq_85_simulation/roboticsgroup_gazebo_plugins/package.xml 	new file:   robotiq_85_gripper/robotiq_85_simulation/roboticsgroup_gazebo_plugins/src/disable_link_plugin.cpp 	new file:   robotiq_85_gripper/robotiq_85_simulation/roboticsgroup_gazebo_plugins/src/mimic_joint_plugin.cpp 	new file:   robotiq_85_gripper/robotiq_85_simulation/robotiq_85_gazebo/CMakeLists.txt 	new file:   robotiq_85_gripper/robotiq_85_simulation/robotiq_85_gazebo/controller/gripper_controller_robotiq.yaml 	new file:   robotiq_85_gripper/robotiq_85_simulation/robotiq_85_gazebo/controller/joint_state_controller.yaml 	new file:   robotiq_85_gripper/robotiq_85_simulation/robotiq_85_gazebo/launch/controller_utils.launch 	new file:   robotiq_85_gripper/robotiq_85_simulation/robotiq_85_gazebo/launch/robotiq_85.launch 	new file:   robotiq_85_gripper/robotiq_85_simulation/robotiq_85_gazebo/launch/robotiq_85_moveit_rviz_test.launch 	new file:   robotiq_85_gripper/robotiq_85_simulation/robotiq_85_gazebo/launch/robotiq_85_moveit_sim.launch 	new file:   robotiq_85_gripper/robotiq_85_simulation/robotiq_85_gazebo/launch/test_kinematics.launch 	new file:   robotiq_85_gripper/robotiq_85_simulation/robotiq_85_gazebo/package.xml 	new file:   robotiq_85_gripper/robotiq_85_simulation/robotiq_85_gazebo/scripts/robotiq_85_moveit_test.py 	new file:   robotiq_85_gripper/robotiq_85_simulation/robotiq_85_simulation/CMakeLists.txt 	new file:   robotiq_85_gripper/robotiq_85_simulation/robotiq_85_simulation/package.xml 	new file:   robotiq_85_gripper/si_utils/CMakeLists.txt 	new file:   robotiq_85_gripper/si_utils/launch/test.launch 	new file:   robotiq_85_gripper/si_utils/package.xml 	new file:   robotiq_85_gripper/si_utils/scripts/timed_roslaunch 	new file:   ur3_with_robotiq_gripper_description/CMakeLists.txt 	new file:   ur3_with_robotiq_gripper_description/launch/ur3_robotiq_upload.launch 	new file:   ur3_with_robotiq_gripper_description/launch/view_ur3_robotiq.launch 	new file:   ur3_with_robotiq_gripper_description/package.xml 	new file:   ur3_with_robotiq_gripper_description/urdf/ur3_robotiq.xacro 	modified:   ur_description/urdf/common.gazebo.xacro 	modified:   ur_description/urdf/ur3.urdf.xacro 	modified:   ur_gazebo/launch/ur3.launch 	new file:   ur_gazebo/worlds/ur3_proyecto.world

File: ur_description/urdf/common.gazebo.xacro (robot description, xacro)
@@ -21,54 +21,36 @@
 -->
   </gazebo>
-  <!-- camera_link -->
-  <gazebo reference="camera_link">
-    <mu1>0.2</mu1>
-    <mu2>0.2</mu2>
-    <material>Gazebo/Green</material>
-  </gazebo>
- <!-- camera -->
-  <gazebo reference="camera_link">
-    <sensor type="camera" name="camera1">
-      <update_rate>30.0</update_rate>
-      <camera name="head">
-        <horizontal_fov>1.3962634</horizontal_fov>
-        <image>
-          <width>800</width>
-          <height>800</height>
-          <format>R8G8B8</format>
-        </image>
-        <clip>
-          <near>0.02</near>
-          <far>300</far>
-        </clip>
+<gazebo reference="hokuyo_link">
+    <sensor type="ray" name="head_hokuyo_sensor">
+      <pose>0 0 0 0 0 0</pose>
+      <visualize>true</visualize>
+      <update_rate>40</update_rate>
+      <ray>
+        <scan>
+          <horizontal>
+            <samples>720</samples>
+            <resolution>1</resolution>
+            <min_angle>-1.570796</min_angle>
+            <max_angle>1.570796</max_angle>
+          </horizontal>
+        </scan>
+        <range>
+          <min>0.10</min>
+          <max>30.0</max>
+          <resolution>0.01</resolution>
+        </range>
         <noise>
           <type>gaussian</type>
-          <!-- Noise is sampled independently per pixel on each frame.
-               That pixel's noise value is added to each of its color
-               channels, which at that point lie in the range [0,1]. -->
+          <!-- Noise parameters based on published spec for Hokuyo laser
+               achieving "+-30mm" accuracy at range < 10m.  A mean of 0.0m and
+               stddev of 0.01m will put 99.7% of samples within 0.03m of the true
+               reading. -->
           <mean>0.0</mean>
-          <stddev>0.007</stddev>
+          <stddev>0.01</stddev>
         </noise>
-      </camera>
-      <plugin name="camera_controller" filename="libgazebo_ros_camera.so">
-        <alwaysOn>true</alwaysOn>
-        <updateRate>0.0</updateRate>
-        <cameraName>ur5/usbcam</cameraName>
-        <imageTopicName>image_raw</imageTopicName>
-        <cameraInfoTopicName>camera_info</cameraInfoTopicName>
-        <frameName>camera_link_optical</frameName>
-        <!-- setting hackBaseline to anything but 0.0 will cause a misalignment
-            between the gazebo sensor image and the frame it is supposed to
-            be attached to -->
-        <hackBaseline>0.0</hackBaseline>
-        <distortionK1>0.0</distortionK1>
-        <distortionK2>0.0</distortionK2>
-        <distortionK3>0.0</distortionK3>
-        <distortionT1>0.0</distortionT1>
-        <distortionT2>0.0</distortionT2>
-        <CxPrime>0</CxPrime>
-        <Cx>0.0</Cx>
-        <Cy>0.0</Cy>
-        <focalLength>0.0</focalLength>
+      </ray>
+      <plugin name="gazebo_ros_head_hokuyo_controller" filename="libgazebo_ros_laser.so">
+        <topicName>/ur3/laser/scan</topicName>
+        <frameName>hokuyo_link</frameName>
       </plugin>
     </sensor>

File: ur_description/urdf/ur3.urdf.xacro (robot description, xacro)
@@ -334,4 +334,19 @@
       <child link="${prefix}tool0"/>
     </joint>
+	<joint name="hokuyo_joint" type="fixed">
+	  <axis xyz="0 1 0" />
+	  <origin xyz="0 0 0" rpy="0 0 0"/>
+	  <parent link="base_link"/>
+	  <child link="hokuyo_link"/>
+	</joint>
+	<!-- Hokuyo Laser -->
+	<link name="hokuyo_link">
+	  <collision>
+		<origin xyz="0 0 0" rpy="0 0 0"/>
+		<geometry>
+	  <box size="0.1 0.1 0.1"/>
+		</geometry>
+	  </collision>
+	</link>
   </xacro:macro>
 </robot>

Commit message: modified:   ur_description/urdf/common.gazebo.xacro 	modified:   ur_description/urdf/ur3.urdf.xacro 	modified:   ur_gazebo/launch/ur3.launch 	modified:   ur_gazebo/worlds/ur3_proyecto.world

File: ur_description/urdf/common.gazebo.xacro (robot description, xacro)
@@ -21,38 +21,3 @@
 -->
   </gazebo>
-<gazebo reference="hokuyo_link">
-    <sensor type="ray" name="head_hokuyo_sensor">
-      <pose>0 0 0 0 0 0</pose>
-      <visualize>true</visualize>
-      <update_rate>40</update_rate>
-      <ray>
-        <scan>
-          <horizontal>
-            <samples>720</samples>
-            <resolution>1</resolution>
-            <min_angle>-1.570796</min_angle>
-            <max_angle>1.570796</max_angle>
-          </horizontal>
-        </scan>
-        <range>
-          <min>0.10</min>
-          <max>30.0</max>
-          <resolution>0.01</resolution>
-        </range>
-        <noise>
-          <type>gaussian</type>
-          <!-- Noise parameters based on published spec for Hokuyo laser
-               achieving "+-30mm" accuracy at range < 10m.  A mean of 0.0m and
-               stddev of 0.01m will put 99.7% of samples within 0.03m of the true
-               reading. -->
-          <mean>0.0</mean>
-          <stddev>0.01</stddev>
-        </noise>
-      </ray>
-      <plugin name="gazebo_ros_head_hokuyo_controller" filename="libgazebo_ros_laser.so">
-        <topicName>/ur3/laser/scan</topicName>
-        <frameName>hokuyo_link</frameName>
-      </plugin>
-    </sensor>
-  </gazebo>
 </robot>

File: ur_description/urdf/ur3.urdf.xacro (robot description, xacro)
@@ -334,19 +334,4 @@
       <child link="${prefix}tool0"/>
     </joint>
-	<joint name="hokuyo_joint" type="fixed">
-	  <axis xyz="0 1 0" />
-	  <origin xyz="0 0 0" rpy="0 0 0"/>
-	  <parent link="base_link"/>
-	  <child link="hokuyo_link"/>
-	</joint>
-	<!-- Hokuyo Laser -->
-	<link name="hokuyo_link">
-	  <collision>
-		<origin xyz="0 0 0" rpy="0 0 0"/>
-		<geometry>
-	  <box size="0.1 0.1 0.1"/>
-		</geometry>
-	  </collision>
-	</link>
   </xacro:macro>
 </robot>
